File: ILJJ_Mk-VII.sch (KiCad schematic (older format))
At the start: 25 parts, among them J1 Conn_02x12, U1 74LS00, U10 74LS00, U11 74LS00, U2 74LS00, U3 74LS00, U4 74LS00, U5 74LS00, U6 74LS00, U7 74LS00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

Commit message: [change] CinとCoutを交換
Changed lines of the file:
@@
 Wire Wire Line
 	1750 3500 1600 3500
+Text Label 1750 2800 2    50   ~ 0
+Cin
 Text Label 950  2800 0    50   ~ 0
-Cin
-Text Label 1750 2800 2    50   ~ 0
 Cout
 Text Label 950  3400 0    50   ~ 0

Commit message: [change] パワーランプの位置を変更
Parts:
- R1: footprint Resistors_ThroughHole:R_Axial_DIN0207_L6.3mm_D2.5mm_P7.62mm_Horizontal -> Resistors_ThroughHole:R_Axial_DIN0207_L6.3mm_D2.5mm_P2.54mm_Vertical
Changed lines of the file:
@@
 F 0 "R1" H 1020 4296 50  0000 L CNN
 F 1 "R" H 1020 4205 50  0000 L CNN
-F 2 "Resistors_ThroughHole:R_Axial_DIN0207_L6.3mm_D2.5mm_P7.62mm_Horizontal" V 880 4250 50  0001 C CNN
+F 2 "Resistors_ThroughHole:R_Axial_DIN0207_L6.3mm_D2.5mm_P2.54mm_Vertical" V 880 4250 50  0001 C CNN
 F 3 "~" H 950 4250 50  0001 C CNN
 	1    950  4250
